File: PCB/_autosave-PCB.kicad_pcb (KiCad board)
At the start: 2 copper layers, 10 parts, among them J1 Screw_Terminal_01x04, J2 Screw_Terminal_01x02, J3 Screw_Terminal_01x02, J5 Conn_01x12_Pin, J6 Conn_01x12_Pin, J7 Screw_Terminal_01x04, J8 Conn_01x04_Pin

Commit message: Lunes 20/01
Parts:
- added J2: Conn_01x16_Socket, Connector_PinHeader_2.00mm:PinHeader_1x16_P2.00mm_Vertical, F.Cu at (151.0, 24.5)
- added J3: Conn_01x17_Pin, Connector_PinSocket_2.54mm:PinSocket_1x17_P2.54mm_Vertical, F.Cu at (108.0, 42.1)
- J5, J6: footprint Connector_PinHeader_2.54mm:PinHeader_1x12_P2.54mm_Vertical -> Connector_PinSocket_2.54mm:PinSocket_1x12_P2.54mm_Vertical
- J8: footprint Connector_PinHeader_2.54mm:PinHeader_1x04_P2.54mm_Vertical -> Connector_PinSocket_2.54mm:PinSocket_1x04_P2.54mm_Vertical
- Je1: footprint Connector_PinHeader_2.54mm:PinHeader_1x06_P2.54mm_Vertical -> Connector_PinSocket_2.54mm:PinSocket_1x06_P2.54mm_Vertical
- moved ArduinoMicro1 24.3 mm to (188.1, 48.3)
- moved Je1 2.24 mm to (146.5, 131.7)
- moved J8 2.24 mm to (149.1, 107.2)
- moved J7 1.50 mm to (189.5, 116.5)
- moved J1 1.41 mm to (145.0, 143.5)
- moved J5 1.12 mm to (195.2, 147.5)
- moved J6 1.12 mm to (195.2, 134.5)
Routing:
- net (no net): track 0.71 -> 0.00 mm
