File: PCB/PCB.kicad_pcb (KiCad board)
At the start: 2 copper layers, 10 parts, among them J1 Screw_Terminal_01x04, J2 Screw_Terminal_01x02, J3 Screw_Terminal_01x02, J5 Conn_01x12_Pin, J6 Conn_01x12_Pin, J7 Screw_Terminal_01x04, J8 Conn_01x04_Pin

Commit message: 28 del 1
Parts:
- removed J7: Screw_Terminal_01x04, TerminalBlock:TerminalBlock_Altech_AK300-4_P5.00mm
- added J2: Conn_01x16_Socket, Connector_PinHeader_2.00mm:PinHeader_1x16_P2.00mm_Vertical, F.Cu at (151.0, 24.5)
- added J2: Screw_Terminal_01x04, TerminalBlock:TerminalBlock_Altech_AK300-4_P5.00mm, F.Cu at (248.0, 71.0)
- added J3: Conn_01x17_Pin, Connector_PinSocket_2.54mm:PinSocket_1x17_P2.54mm_Vertical, F.Cu at (108.0, 42.1)
- added J4: Conn_01x04_Pin, Connector_PinHeader_2.54mm:PinHeader_1x04_P2.54mm_Vertical, F.Cu at (218.0, 102.8)
- J5, J6: footprint Connector_PinHeader_2.54mm:PinHeader_1x12_P2.54mm_Vertical -> Connector_PinSocket_2.54mm:PinSocket_1x12_P2.54mm_Vertical
- J8: footprint Connector_PinHeader_2.54mm:PinHeader_1x04_P2.54mm_Vertical -> Connector_PinSocket_2.54mm:PinSocket_1x04_P2.54mm_Vertical
- Je1: footprint Connector_PinHeader_2.54mm:PinHeader_1x06_P2.54mm_Vertical -> Connector_PinSocket_2.54mm:PinSocket_1x06_P2.54mm_Vertical
- moved J8 101.2 mm to (247.0, 87.0)
- moved Je1 101.2 mm to (244.4, 111.5)
- moved J1 90.6 mm to (232.7, 124.0)
- moved J5 68.7 mm to (223.5, 84.1), turned to 0 degrees
- moved J6 65.0 mm to (236.5, 83.8), turned to 0 degrees
- moved ArduinoMicro1 24.3 mm to (188.1, 48.3)
Connections:
- J5 pad 3: unconnected-(J5-Pin_3-Pad3) -> GND
- J5 pad 4: unconnected-(J5-Pin_4-Pad4) -> GND
- J6 pad 10: unconnected-(J6-Pin_10-Pad10) -> Net-(J6-Pin_10)
- J6 pad 11: Net-(J6-Pin_11) -> unconnected-(J6-Pin_11-Pad11)
- J6 pad 12: Net-(J6-Pin_12) -> unconnected-(J6-Pin_12-Pad12)
- J6 pad 2: Net-(J6-Pin_2) -> GND
- J6 pad 9: unconnected-(J6-Pin_9-Pad9) -> Net-(J6-Pin_9)
- J8 pad 1: Net-(J6-Pin_2) -> GND
- J8 pad 2: Net-(J6-Pin_12) -> Net-(J6-Pin_9)
- J8 pad 3: Net-(J6-Pin_11) -> Net-(J6-Pin_10)
Routing:
- net Net-(J1-Pin_2): track 0.00 -> 129.3 mm
- net Net-(J1-Pin_3): track 0.00 -> 105.5 mm
- net Net-(J1-Pin_1): track 0.00 -> 82.2 mm
- net Net-(J1-Pin_4): track 0.00 -> 63.0 mm
- net Net-(J4-Pin_4): track 0.00 -> 50.8 mm
- net Net-(J6-Pin_10): track 0.00 -> 27.5 mm
- net Net-(J6-Pin_9): track 0.00 -> 24.6 mm
- net Net-(J4-Pin_3): track 0.00 -> 16.9 mm
- net Net-(J4-Pin_2): track 0.00 -> 15.9 mm
- added copper zone on F.Cu, net GND
