File: .kikad/Pico_4hx_ori/Pico_4hx.kicad_pcb (KiCad board)
At the start: 2 copper layers, 18 parts, among them J1 Conn_01x48_Pin, J7 USB_A, U1 Pico

Commit message: Control
Parts:
- removed the ? at (273.6, 59.5)
- removed the ? at (159.6, 59.5)
- removed the ? at (159.1, 121.0)
- removed the ? at (274.1, 121.0)
- added ?: , , F.Cu at (158.5, 120.1)
- added ?: , , F.Cu at (278.3, 59.4)
- added ?: , , F.Cu at (278.3, 120.1)
- added ?: , , F.Cu at (158.5, 59.4)
- moved ? 5.97 mm to (253.5, 105.7)
- moved U1 5.97 mm to (256.2, 81.2)
- moved ? 5.97 mm to (258.7, 105.7)
- moved J7 5.97 mm to (252.5, 111.5)
- moved J1 1.42 mm to (223.2, 119.9)
Routing:
- net DT1: track 74.9 -> 86.7 mm
- net VCC: track 110.1 -> 118.8 mm
- net DT2: track 59.6 -> 66.1 mm
- net DT3: track 39.3 -> 45.2 mm
- net DT4: track 19.2 -> 24.4 mm
- net SCK: track 98.4 -> 103.6 mm
- net 4A+: track 32.5 -> 30.9 mm
- net 1A-: track 47.5 -> 46.0 mm
- net 4A-: track 42.8 -> 41.4 mm
- net 3A-: track 43.5 -> 42.0 mm
- net 3A+: track 32.0 -> 30.5 mm
- net 1E+: track 57.4 -> 55.9 mm
- net 4E+: track 51.7 -> 50.3 mm
- net 3E+: track 52.9 -> 51.4 mm
- net 2E+: track 53.7 -> 52.3 mm
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