File: .kikad/ProPico-main/ProPico.kicad_pcb (KiCad board)
At the start: 2 copper layers, 96 parts, among them J1 USB_C_Receptacle_USB2.0, J2 SWD, SW1 BOOTSEL, SW2 RES, U1 FM24CL16B, U10 HX711, U11 MMBT5550LT1G, U12 HX711, U13 MMBT5550LT1G, U14 HX711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

Commit message: Control
Parts:
- removed G***: LOGO, LOGO
- removed HX4_C2, HX_C1, HX_C3: 0.1uF, Capacitor_SMD:C_1206_3216Metric
- removed HX5_C5, HX_C4, HX_C5: 10uF, Capacitor_SMD:C_1206_3216Metric
- removed HX_R1: 20k, Resistor_SMD:R_1206_3216Metric
- removed HX_R2: 8.2k, Resistor_SMD:R_1206_3216Metric
- removed HX_R3: 1k, Resistor_SMD:R_1206_3216Metric
- removed J1: USB_C_Receptacle_USB2.0, Connector_USB:USB_C_Receptacle_Palconn_UTC16-G
- removed TP4: GND, TestPoint:TestPoint_Pad_1.5x1.5mm
- removed TP5: D+, TestPoint:TestPoint_Pad_1.5x1.5mm
- removed TP7: D-, TestPoint:TestPoint_Pad_1.5x1.5mm
- removed U10, U12, U14, U9: HX711, Package_SO:SOP-16_3.9x9.9mm_P1.27mm
- removed U11, U13, U7, U8: MMBT5550LT1G, Package_TO_SOT_SMD:TSOT-23
- added C19: 0.1uF, Capacitor_SMD:C_0805_2012Metric_Pad1.18x1.45mm_HandSolder, F.Cu at (140.9, 80.8)
- added C20: 0.1uF, Capacitor_SMD:C_0805_2012Metric_Pad1.18x1.45mm_HandSolder, F.Cu at (129.6, 80.8)
- added HX1_C1: 0.1uF, Capacitor_SMD:C_1206_3216Metric, F.Cu at (128.5, 59.4)
- added HX1_C3: 0.1uF, Capacitor_SMD:C_1206_3216Metric, F.Cu at (120.5, 57.9)
- added HX1_C4: 10uF, Capacitor_SMD:C_1206_3216Metric, F.Cu at (129.2, 53.9)
- added HX1_C5: 10uF, Capacitor_SMD:C_1206_3216Metric, F.Cu at (118.1, 46.2)
- added HX1_R1: 20k, Resistor_SMD:R_1206_3216Metric, F.Cu at (120.4, 62.8)
- added HX1_R2: 8.2k, Resistor_SMD:R_1206_3216Metric, F.Cu at (123.0, 62.8)
- added HX1_R3: 1k, Resistor_SMD:R_1206_3216Metric, F.Cu at (128.5, 62.6)
- added HX4_C1: 0.1uF, Capacitor_SMD:C_1206_3216Metric, F.Cu at (68.5, 59.4)
- added HX4_C5: 10uF, Capacitor_SMD:C_1206_3216Metric, F.Cu at (58.1, 46.2)
- added HX711_1: HX711, Package_SO:SOP-16_3.9x9.9mm_P1.27mm, F.Cu at (121.1, 52.4)
- added HX711_2: HX711, Package_SO:SOP-16_3.9x9.9mm_P1.27mm, F.Cu at (101.1, 52.4)
- added HX711_3: HX711, Package_SO:SOP-16_3.9x9.9mm_P1.27mm, F.Cu at (81.1, 52.4)
- added HX711_4: HX711, Package_SO:SOP-16_3.9x9.9mm_P1.27mm, F.Cu at (61.1, 52.4)
- added J5: 74355-1042LF, Connector_Amphenol:NCR_PIN_AMPHENOL_74355-1042LF, F.Cu at (153.2, 81.1)
- added TR1: MMBT5550LT1G, Package_TO_SOT_SMD:TSOT-23, F.Cu at (116.0, 60.5)
- added TR2: MMBT5550LT1G, Package_TO_SOT_SMD:TSOT-23, F.Cu at (96.0, 60.5)
- added TR3: MMBT5550LT1G, Package_TO_SOT_SMD:TSOT-23, F.Cu at (76.0, 60.5)
- added TR4: MMBT5550LT1G, Package_TO_SOT_SMD:TSOT-23, F.Cu at (56.0, 60.5)
- moved LM1 29.4 mm to (135.4, 86.2), turned to 180 degrees
- moved D1 15.0 mm to (138.9, 67.5), turned to 180 degrees
- moved C1 6.25 mm to (156.1, 39.6)
- moved C15 6.25 mm to (153.8, 58.4)
- moved C18 6.25 mm to (153.1, 45.2)
- moved R10 6.25 mm to (153.5, 40.7)
- moved R3 6.25 mm to (156.1, 68.2)
- moved R4 6.25 mm to (150.8, 68.2)
- moved R5 6.25 mm to (154.6, 44.1)
- moved U5 6.25 mm to (153.2, 51.5)
- moved C4 6.25 mm to (147.6, 68.5)
- moved D3 6.25 mm to (159.0, 68.5)
- moved TP6 6.25 mm to (155.7, 68.9)
- moved C10 6.25 mm to (149.4, 57.7)
- moved C12 6.25 mm to (148.4, 57.7)
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Connections:
- HX2_C1 pad 2: (no net) -> Net-(HX711_2-INA+)
- HX2_C4 pad 1: (no net) -> Net-(HX711_2-VBG)
- HX2_R1 pad 2: (no net) -> Net-(HX711_2-VFB)
- HX2_R2 pad 2: (no net) -> Net-(HX711_2-VFB)
- HX2_R3 pad 2: (no net) -> Net-(HX711_2-INA+)
- HX3_C1 pad 2: (no net) -> Net-(HX711_3-INA+)
- HX3_C4 pad 1: (no net) -> Net-(HX711_3-VBG)
- HX3_R1 pad 2: (no net) -> Net-(HX711_3-VFB)
- HX3_R2 pad 2: (no net) -> Net-(HX711_3-VFB)
- HX3_R3 pad 2: (no net) -> Net-(HX711_3-INA+)
- HX4_C4 pad 1: (no net) -> Net-(HX711_4-VBG)
- HX4_R1 pad 2: (no net) -> Net-(HX711_4-VFB)
- HX4_R2 pad 2: (no net) -> Net-(HX711_4-VFB)
- HX4_R3 pad 2: (no net) -> Net-(HX711_4-INA+)
- LM1 pad 1: unconnected-(LM1-INPUT-Pad1) -> Net-(LM1-INPUT)
- LM1 pad 2: unconnected-(LM1-GROUND-Pad2) -> GND
- LM1 pad 3: unconnected-(LM1-OUTPUT-Pad3) -> VBUS
Routing:
- net (no net): track 67.7 -> 0.00 mm
- net 3.3V: track 210.2 -> 275.4 mm
- net SDA4: track 92.7 -> 31.5 mm
- net SDA3: track 80.3 -> 24.3 mm
- net SCL: track 151.0 -> 192.4 mm
- net Net-(LM1-INPUT): track 0.00 -> 25.7 mm, vias 0 -> 1
- net VBUS: track 0.00 -> 18.0 mm
- net 2E+: track 42.1 -> 31.6 mm
- net Net-(U9-INA+): track 10.1 -> 0.00 mm
- net Net-(HX711_1-INA+): track 0.00 -> 10.1 mm
- net Net-(HX711_4-INA+): track 0.00 -> 10.1 mm
- net Net-(HX711_3-INA+): track 0.00 -> 10.1 mm
- net Net-(HX711_2-INA+): track 0.00 -> 10.1 mm
- net /D+: track 21.6 -> 12.1 mm, vias 1 -> 0
- net Net-(HX711_3-VFB): track 0.00 -> 9.30 mm
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- removed copper zone on F.Cu, net VBUS
- removed copper zone on F.Cu, net VCC
Other:
- board text added: "Scale by Girboy"
- board text removed: "PRO PICO by diminDDL"
