File: .kikad/ProPico-main/ProPico.kicad_sch (KiCad schematic)
At the start: 93 parts, among them J1 USB_C_Receptacle_USB2.0, J2 SWD, J3 LEFT, J4 RIGHT, SW1 BOOTSEL, SW2 RES, U1 FM24CL16B, U10 HX711, U11 MMBT5550LT1G, U12 HX711, U13 MMBT5550LT1G, U14 HX711, U2 W25Q16JVUXIQ, U3 AMS1117-3.3, U4 LM4040DBZ-3, U5 RP2040, U6 MMBT5550LT1G, U7 MMBT5550LT1G, U9 HX711, Y1 ECS-120-12-36-AGN-TR3

Commit message: Control
Parts:
- removed U10, U12, U14: HX711, Package_SO:SOP-16_3.9x9.9mm_P1.27mm, symbol Analog_ADC:HX711
- removed U11, U13, U7: MMBT5550LT1G, Package_TO_SOT_SMD:TSOT-23, symbol S9015:MMBT5550LT1G
- added C19, C20: 0.1uF, Capacitor_SMD:C_0805_2012Metric_Pad1.18x1.45mm_HandSolder, symbol Device:C
- added HX711_2, HX711_3, HX711_4: HX711, Package_SO:SOP-16_3.9x9.9mm_P1.27mm, symbol Analog_ADC:HX711
- added J5: 74355-1042LF, Connector_Amphenol:NCR_PIN_AMPHENOL_74355-1042LF, symbol NCR PIN:74355-1042LF
- added TR2, TR3, TR4: MMBT5550LT1G, Package_TO_SOT_SMD:TSOT-23, symbol S9015:MMBT5550LT1G
- HX2_C3, HX3_C3, HX4_C3: value 10uF -> 0.1uF
- HX2_C4, HX3_C4, HX4_C4: value 0.1uF -> 10uF
- HX2_R1, HX3_R1, HX4_R1: value 1k -> 20k
- HX2_R3, HX3_R3, HX4_R3: value 20k -> 1k
- renumbered HX_C1 to HX1_C1, HX_C4 to HX1_C3, HX_C3 to HX1_C4, HX_C5 to HX1_C5, HX_R3 to HX1_R1, HX_R2 to HX1_R2, HX_R1 to HX1_R3, U9 to HX711_1, U6 to TR1
Connections:
- net GPIO28_ADC2 is gone; now on net SDA4: J4.14 (Pin_14), U5.40 (GPIO28_ADC2)
- net GPIO29_ADC3 is gone; now on net SDA3: J4.17 (Pin_17), U5.41 (GPIO29_ADC3)
- net +5V: now also HX711_2.1 (VSUP), HX711_2.15 (RATE), HX711_2.16 (DVDD), HX711_3.1 (VSUP), HX711_3.15 (RATE), HX711_3.16 (DVDD), HX711_4.1 (VSUP), HX711_4.15 (RATE), HX711_4.16 (DVDD), TR2.2 (EMITTER), TR3.2 (EMITTER), TR4.2 (EMITTER)
- net 2A+: now also HX2_R3.1; no longer HX2_R1.1
- net 2A-: now also HX711_2.7 (INA-)
- net 2E+: now also HX2_C3.1, HX2_R1.1, HX711_2.3 (AVDD), TR2.3 (COLLECTOR); no longer HX2_C4.1, HX2_R3.1
- net 2E-: now also HX711_2.5 (AGND)
- net 3A+: now also HX3_R3.1; no longer HX3_R1.1
- net 3A-: now also HX711_3.7 (INA-)
- net 3E+: now also HX3_C3.1, HX3_R1.1, HX711_3.3 (AVDD), TR3.3 (COLLECTOR); no longer HX3_C4.1, HX3_R3.1
- net 3E-: now also HX711_3.5 (AGND)
- net 4A+: now also HX4_R3.1; no longer HX4_R1.1
- net 4A-: now also HX711_4.7 (INA-)
- net 4E+: now also HX4_C3.1, HX4_R1.1, HX711_4.3 (AVDD), TR4.3 (COLLECTOR); no longer HX4_C4.1, HX4_R3.1
- net 4E-: now also HX711_4.5 (AGND)
- net DT2: now also HX711_2.12 (DOUT)
- net DT3: now also HX711_3.12 (DOUT)
- net DT4: now also HX711_4.12 (DOUT)
- net GND: now also LM1.2 (GROUND), C19.2, C20.2, HX711_2.14 (XI), HX711_3.14 (XI), HX711_4.14 (XI), J5.4, J5.6, J5.8, J5.G1 (GND), J5.G2 (GND), J5.G3 (GND), J5.G4 (GND), J5.S1 (SHIELD), J5.S2 (SHIELD)
- net SCK: now also HX711_2.11 (PD_SCK), HX711_3.11 (PD_SCK), HX711_4.11 (PD_SCK)
- net VBUS: now also LM1.3 (OUTPUT), C20.1
- net at HX3_R1.2: now also HX3_R2.2, HX711_3.4 (VFB); no longer HX3_C1.2
- net at HX3_R3.2: now also HX3_C1.2, HX711_3.8 (INA+); no longer HX3_R2.2
- net at HX2_R3.2: now also HX2_C1.2, HX711_2.8 (INA+); no longer HX2_R2.2
- net at LM1.1 (INPUT): now also C19.1, J5.3, J5.5
- net at HX2_R1.2: now also HX2_R2.2, HX711_2.4 (VFB); no longer HX2_C1.2
- net at HX4_R3.2: now also HX4_C1.2, HX711_4.8 (INA+); no longer HX4_R2.2
- net at HX4_R1.2: now also HX4_R2.2, HX711_4.4 (VFB); no longer HX4_C1.2
- new net: HX2_C4.1, HX711_2.6 (VBG)
- new net: HX711_3.2 (BASE), TR3.1 (BASE)
- new net: HX3_C4.1, HX711_3.6 (VBG)
- new net: HX711_2.2 (BASE), TR2.1 (BASE)
- new net: HX711_4.2 (BASE), TR4.1 (BASE)
- new net: HX4_C4.1, HX711_4.6 (VBG)
Other:
- moved on the sheet: LM1
