File: .kikad/ProPico-main_ mio/ProPico-main/ProPico.kicad_pcb (KiCad board)
At the start: 2 copper layers, 127 x 71 mm, 96 parts, among them J1 USB_C_Receptacle_USB2.0, J2 SWD, SW1 BOOTSEL, SW2 RES, U1 FM24CL16B, U10 HX711, U11 MMBT5550LT1G, U12 HX711, U13 MMBT5550LT1G, U14 HX711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

Commit message: Control
Parts:
- removed G***: LOGO, LOGO
Routing:
- net 4A+: track 18.4 -> 19.2 mm
- net 4A-: track 26.2 -> 26.9 mm
- net 1A+: track 31.1 -> 31.6 mm
